Commit message: update with acutal robot model dimension & contain launch file for launching the whole system

File: robot_system/urdf/wro_actual.urdf.xacro (robot description, xacro)
@@ -24,11 +24,11 @@
   <xacro:property name="lidar_pos_y" value="0.0"/>    <!-- Centered in y-axis -->
   <xacro:property name="lidar_pos_z" value="0.0456"/>   <!-- 7.5 cm above the base -->
-  <xacro:property name="camera_length" value="0.02"/>   <!-- 25 mm -->
+  <xacro:property name="camera_length" value="0.021"/>   <!-- 25 mm -->
   <xacro:property name="camera_width" value="0.03"/>    <!-- 24 mm -->
   <xacro:property name="camera_height" value="0.03"/>   <!-- 9 mm -->
-  <xacro:property name="camera_pos_x" value="-0.006"/>   <!-- 8.7 cm forward -->
+  <xacro:property name="camera_pos_x" value="-0.002"/>   <!-- 8.7 cm forward -->
   <xacro:property name="camera_pos_y" value="0.0"/>      <!-- Centered in y-axis -->
-  <xacro:property name="camera_pos_z" value="0.09265"/>     <!-- 18.0 cm above base -->
-  <xacro:property name="camera_pitch" value="0.209"/>  <!-- 12 degrees in radians -->
+  <xacro:property name="camera_pos_z" value="0.1106"/>     <!-- 18.0 cm above base -->
+  <xacro:property name="camera_pitch" value="0.262"/>  <!-- 12 degrees in radians -->
   <!-- Base Link -->
   <link name="base_link" />

Commit message: packages updated

File: robot_system/urdf/wro_actual.urdf.xacro (robot description, xacro)
@@ -31,4 +31,5 @@
   <xacro:property name="camera_pos_z" value="0.1106"/>     <!-- 18.0 cm above base -->
   <xacro:property name="camera_pitch" value="0.262"/>  <!-- 12 degrees in radians -->
+  <xacro:property name="camera_yaw" value="-0.05"/>  <!-- 12 degrees in radians -->
   <!-- Base Link -->
   <link name="base_link" />
@@ -253,5 +254,5 @@
     <child link="camera_link"/>
     <!-- Position and orientation for the camera relative to the lidar -->
-    <origin xyz="${camera_pos_x} ${camera_pos_y} ${camera_pos_z}" rpy="0 ${camera_pitch} 0"/>
+    <origin xyz="${camera_pos_x} ${camera_pos_y} ${camera_pos_z}" rpy="0 ${camera_pitch} ${camera_yaw}"/>
   </joint>
 </robot>

Commit message: Update wro_actual.urdf.xacro

File: robot_system/urdf/wro_actual.urdf.xacro (robot description, xacro)
@@ -27,9 +27,9 @@
   <xacro:property name="camera_width" value="0.03"/>    <!-- 24 mm -->
   <xacro:property name="camera_height" value="0.03"/>   <!-- 9 mm -->
-  <xacro:property name="camera_pos_x" value="-0.002"/>   <!-- 8.7 cm forward -->
+  <xacro:property name="camera_pos_x" value="0.03"/>   <!-- 8.7 cm forward -->
   <xacro:property name="camera_pos_y" value="0.0"/>      <!-- Centered in y-axis -->
-  <xacro:property name="camera_pos_z" value="0.1106"/>     <!-- 18.0 cm above base -->
-  <xacro:property name="camera_pitch" value="0.262"/>  <!-- 12 degrees in radians -->
-  <xacro:property name="camera_yaw" value="-0.05"/>  <!-- 12 degrees in radians -->
+  <xacro:property name="camera_pos_z" value="0.10"/>     <!-- 18.0 cm above base -->
+  <xacro:property name="camera_pitch" value="0.191986"/>  <!-- 12 degrees in radians -->
+  <xacro:property name="camera_yaw" value="0.05"/>  <!-- 12 degrees in radians -->
   <!-- Base Link -->
   <link name="base_link" />
